File: schematics/voice/shmoergh-funk-live-voice.kicad_sch (KiCad schematic)
At the start: 25 parts, among them Q1 2N3906, U2 TL074, U4 TL074

Commit message: Added a couple of test points
Parts:
- added TP_AMP_COMP2, TP_RESET1, TP_SAW_BIAS1, TP_SAW_OUT1, TP_SQR_OUT2: TestPoint, symbol Connector:TestPoint
Connections:
- net SAW_OUT: now also TP_SAW_OUT1.1
- net SQR_OUT: now also TP_SQR_OUT2.1
- net at C2.1, R5.1, R7.2: now also TP_RESET1.1
- net at RV_SAW_BIAS1.2, U2.10 (+): now also TP_SAW_BIAS1.1
- net at C1.1, R1.1, U2.5 (+): now also TP_AMP_COMP2.1
Changed lines of the file:
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@@
   (junction (at 158.75 77.47) (diameter 0) (color 0 0 0 0)
+  )
+  (junction (at 173.99 82.55) (diameter 0) (color 0 0 0 0)
   )
   (junction (at 35.56 176.53) (diameter 0) (color 0 0 0 0)
@@
     (stroke (width 0) (type default))
   )
+  (wire (pts (xy 193.04 80.01) (xy 193.04 87.63))
+    (stroke (width 0) (type default))
+  )
   (wire (pts (xy 158.75 127) (xy 158.75 130.81))
     (stroke (width 0) (type default))
@@
   )
   (wire (pts (xy 158.75 113.03) (xy 158.75 119.38))
+    (stroke (width 0) (type default))
+  )
+  (wire (pts (xy 171.45 88.9) (xy 171.45 82.55))
+    (stroke (width 0) (type default))
+  )
+  (wire (pts (xy 95.25 69.85) (xy 95.25 72.39))
+    (stroke (width 0) (type default))
+  )
+  (wire (pts (xy 166.37 88.9) (xy 171.45 88.9))
     (stroke (width 0) (type default))
   )
@@
     (stroke (width 0) (type default))
   )
+  (wire (pts (xy 196.85 128.27) (xy 196.85 133.35))
+    (stroke (width 0) (type default))
+  )
   (wire (pts (xy 154.94 44.45) (xy 158.75 44.45))
     (stroke (width 0) (type default))
@@
     (stroke (width 0) (type default))
   )
+  (wire (pts (xy 128.27 29.21) (xy 128.27 33.02))
+    (stroke (width 0) (type default))
+  )
   (wire (pts (xy 246.38 44.45) (xy 251.46 44.45))
     (stroke (width 0) (type default))
@@
   )
   (wire (pts (xy 123.19 33.02) (xy 128.27 33.02))
+    (stroke (width 0) (type default))
+  )
+  (wire (pts (xy 171.45 82.55) (xy 173.99 82.55))
     (stroke (width 0) (type default))
   )
@@
     (effects (font (size 1.27 1.27)) (justify left bottom))
   )
-  (text "Output aplification A = 1+1 = 2\nto have 6.6Vpp" (at 193.04 87.63 0)
+  (text "Output aplification A = 1+1 = 2\nto have 6.6Vpp" (at 199.39 86.36 0)
     (effects (font (size 1.27 1.27)) (justify left bottom))
   )
@@
   )
   (text "Discharge RC = 10k * 470pF = 4.7us\nCould go with 560p too"
-    (at 99.06 22.86 0)
+    (at 116.84 19.05 0)
     (effects (font (size 1.27 1.27)) (justify left bottom))
   )
@@
     )
   )
+  (symbol (lib_id "Connector:TestPoint") (at 128.27 29.21 0) (unit 1)
+    (in_bom yes) (on_board yes) (dnp no)
+    (property "Reference" "TP_RESET1" (at 130.81 25.4 0)
+      (effects (font (size 1.27 1.27)) (justify left))
+    )
+    (property "Value" "TestPoint" (at 130.81 27.94 0)
+      (effects (font (size 1.27 1.27)) (justify left))
+    )
+    (property "Footprint" "" (at 133.35 29.21 0)
+      (effects (font (size 1.27 1.27)) hide)
+    )
+    (property "Datasheet" "~" (at 133.35 29.21 0)
+      (effects (font (size 1.27 1.27)) hide)
+    )
+    (pin "1")
+    (instances
+      (project "shmoergh-funk-live-voice"
+        (path "/5a9d7fcc-2f93-4fa9-a3de-a561cb7522b6"
+          (reference "TP_RESET1") (unit 1)
+        )
+      )
+    )
+  )
+  (symbol (lib_id "Connector:TestPoint") (at 193.04 87.63 180) (unit 1)
+    (in_bom yes) (on_board yes) (dnp no) (fields_autoplaced)
+    (property "Reference" "TP_SAW_OUT1" (at 195.58 90.297 0)
+      (effects (font (size 1.27 1.27)) (justify right))
+    )
+    (property "Value" "TestPoint" (at 195.58 92.837 0)
+      (effects (font (size 1.27 1.27)) (justify right))
+    )
+    (property "Footprint" "" (at 187.96 87.63 0)
+      (effects (font (size 1.27 1.27)) hide)
+    )
+    (property "Datasheet" "~" (at 187.96 87.63 0)
+      (effects (font (size 1.27 1.27)) hide)
+    )
+    (pin "1")
+    (instances
+      (project "shmoergh-funk-live-voice"
+        (path "/5a9d7fcc-2f93-4fa9-a3de-a561cb7522b6"
+          (reference "TP_SAW_OUT1") (unit 1)
+        )
+      )
+    )
+  )
   (symbol (lib_id "power:GND") (at 196.85 147.32 0) (unit 1)
     (in_bom yes) (on_board yes) (dnp no)
@@
   (symbol (lib_id "Device:R") (at 137.16 33.02 270) (unit 1)
     (in_bom yes) (on_board yes) (dnp no)
-    (property "Reference" "R7" (at 137.16 27.7622 90)
-      (effects (font (size 1.27 1.27)))
-    )
-    (property "Value" "1k" (at 137.16 30.0736 90)
+    (property "Reference" "R7" (at 138.43 35.56 90)
+      (effects (font (size 1.27 1.27)))
+    )
+    (property "Value" "1k" (at 138.43 38.1 90)
       (effects (font (size 1.27 1.27)))
     )
@@
     )
   )
+  (symbol (lib_id "Connector:TestPoint") (at 166.37 88.9 90) (unit 1)
+    (in_bom yes) (on_board yes) (dnp no) (fields_autoplaced)
+    (property "Reference" "TP_SAW_BIAS1" (at 163.068 83.82 90)
+      (effects (font (size 1.27 1.27)))
+    )
+    (property "Value" "TestPoint" (at 163.068 86.36 90)
+      (effects (font (size 1.27 1.27)))
+    )
+    (property "Footprint" "" (at 166.37 83.82 0)
+      (effects (font (size 1.27 1.27)) hide)
+    )
+    (property "Datasheet" "~" (at 166.37 83.82 0)
+      (effects (font (size 1.27 1.27)) hide)
+    )
+    (pin "1")
+    (instances
+      (project "shmoergh-funk-live-voice"
+        (path "/5a9d7fcc-2f93-4fa9-a3de-a561cb7522b6"
+          (reference "TP_SAW_BIAS1") (unit 1)
+        )
+      )
+    )
+  )
   (symbol (lib_id "Amplifier_Operational:TL074") (at 172.72 133.35 0) (mirror x) (unit 4)
     (in_bom yes) (on_board yes) (dnp no)
@@
     )
   )
+  (symbol (lib_id "Connector:TestPoint") (at 196.85 128.27 0) (unit 1)
+    (in_bom yes) (on_board yes) (dnp no) (fields_autoplaced)
+    (property "Reference" "TP_SQR_OUT2" (at 199.39 124.333 0)
+      (effects (font (size 1.27 1.27)) (justify left))
+    )
+    (property "Value" "TestPoint" (at 199.39 126.873 0)
+      (effects (font (size 1.27 1.27)) (justify left))
+    )
+    (property "Footprint" "" (at 201.93 128.27 0)
+      (effects (font (size 1.27 1.27)) hide)
+    )
+    (property "Datasheet" "~" (at 201.93 128.27 0)
+      (effects (font (size 1.27 1.27)) hide)
+    )
+    (pin "1")
+    (instances
+      (project "shmoergh-funk-live-voice"
+        (path "/5a9d7fcc-2f93-4fa9-a3de-a561cb7522b6"
+          (reference "TP_SQR_OUT2") (unit 1)
+        )
+      )
+    )
+  )
   (symbol (lib_id "Device:R") (at 130.81 74.93 270) (unit 1)
     (in_bom yes) (on_board yes) (dnp no)
@@
         )
       )
+    )
+  )
+  (symbol (lib_id "Connector:TestPoint") (at 95.25 69.85 0) (unit 1)
+    (in_bom yes) (on_board yes) (dnp no) (fields_autoplaced)
+    (property "Reference" "TP_AMP_COMP2" (at 97.79 65.913 0)
+      (effects (font (size 1.27 1.27)) (justify left))
+    )
+    (property "Value" "TestPoint" (at 97.79 68.453 0)
+      (effects (font (size 1.27 1.27)) (justify left))
+    )
+    (property "Footprint" "" (at 100.33 69.85 0)
+      (effects (font (size 1.27 1.27)) hide)
+    )
+    (property "Datasheet" "~" (at 100.33 69.85 0)
+      (effects (font (size 1.27 1.27)) hide)
+    )
+    (pin "1")
+    (instances
+      (project "shmoergh-funk-live-voice"
+        (path "/5a9d7fcc-2f93-4fa9-a3de-a561cb7522b6"
+          (reference "TP_AMP_COMP2") (unit 1)
+        )
+      )
