File: 1.1/schematics/control/shmoergh-funk-live-control.kicad_pcb (KiCad board)
At the start: 2 copper layers, 242.5 x 102.5 mm, 162 parts, among them J1 Power, J2 Power, J3 Power, J4 Power, J5 Power, J6 Power, Q1 BC548C, Q2 BC558, Q3 BC548, Q4 BC548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

Commit message: ✨ 1.1 Release
Hardware
- Fixes missing capacitor on the inputs of mixers. At f=0Hz the DCO's produce a DC output which shifts the center point of DCO's where f>0Hz. This happens on both the sawtooth and the squarewave output. A 470nF foil capacitor blocks all DC input on the input of the mixers.
- Decreases the aplification of mixers. The sum of 6 voices on both saw and square mixers are way too strong and hit the op-amp limits (+/-12V). The first stage of the mixers are reduced now to 1/3 on the squarewave and 1/2 on the sawtooth. Sounds much smoother!

Software
- Updates the MUX and the amp compensation output pin numbers according to the schematics.
Parts:
- added C27: 470n (foil), Capacitor_THT:C_Rect_L7.0mm_W3.5mm_P5.00mm, F.Cu at (182.5, 117.0)
- added C28: 470n (foil), Capacitor_THT:C_Rect_L7.0mm_W3.5mm_P5.00mm, F.Cu at (178.3, 132.3)
- R20: value 100k -> 47k
- R21: value 100k -> 33k
- moved R13 2.92 mm to (186.1, 110.0)
- moved R19 2.92 mm to (189.2, 110.0)
Connections:
- R10 pad 2: Net-(U6A--) -> Net-(C27-Pad1)
- R11 pad 2: Net-(U6A--) -> Net-(C27-Pad1)
- R12 pad 2: Net-(U6A--) -> Net-(C27-Pad1)
- R13 pad 2: Net-(U6A--) -> Net-(C27-Pad1)
- R14 pad 2: Net-(U6C--) -> Net-(C28-Pad1)
- R15 pad 2: Net-(U6C--) -> Net-(C28-Pad1)
- R16 pad 2: Net-(U6C--) -> Net-(C28-Pad1)
- R17 pad 2: Net-(U6C--) -> Net-(C28-Pad1)
- R18 pad 2: Net-(U6C--) -> Net-(C28-Pad1)
- R19 pad 2: Net-(U6C--) -> Net-(C28-Pad1)
- R8 pad 2: Net-(U6A--) -> Net-(C27-Pad1)
- R9 pad 2: Net-(U6A--) -> Net-(C27-Pad1)
Routing:
- net Net-(U6C--): track 152.2 -> 33.8 mm, vias 4 -> 2
- net Net-(C28-Pad1): track 0.00 -> 112.1 mm, vias 0 -> 1
- net Net-(U6A--): track 109.1 -> 15.2 mm, vias 2 -> 1
- net Net-(C27-Pad1): track 0.00 -> 89.0 mm
- net /Mixer/SAW_6_IN: track 14.1 -> 11.1 mm
- net /Mixer/SQR_6_IN: track 9.77 -> 6.85 mm
- net -12V: track 673.6 -> 675.2 mm
- net Net-(C4-Pad2): track 25.9 -> 26.8 mm
Other:
- board text added: "Shmøergh - Sometimes we deliver on time!"
- board text added: "Version 1.1 https://github.com/peterzimon/shmoergh-funk-live"
- board text removed: "Shmøergh - Almost good!"
