File: 1.1/schematics/control/shmoergh-funk-live-control.kicad_sch (KiCad schematic)
At the start: 9 parts

Commit message: 1.1 changes
Other:
- sheet Digital ports: added EXTRA_ADC; removed none
- sheet Filter Interface ports: added FILTER_POSITION; removed none
Changed lines of the file:
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@@
   (junction (at 92.71 111.76) (diameter 0) (color 0 0 0 0)
   )
-  (wire (pts (xy 53.34 58.42) (xy 68.58 58.42))
+  (wire (pts (xy 49.53 58.42) (xy 68.58 58.42))
     (stroke (width 0) (type default))
   )
@@
     (stroke (width 0) (type default))
   )
-  (wire (pts (xy 53.34 45.72) (xy 78.74 45.72))
+  (wire (pts (xy 49.53 45.72) (xy 78.74 45.72))
     (stroke (width 0) (type default))
   )
@@
     (stroke (width 0) (type default))
   )
+  (wire (pts (xy 49.53 76.2) (xy 53.34 76.2))
+    (stroke (width 0) (type default))
+  )
   (wire (pts (xy 55.88 148.59) (xy 198.12 148.59))
     (stroke (width 0) (type default))
@@
     (stroke (width 0) (type default))
   )
-  (wire (pts (xy 53.34 33.02) (xy 95.25 33.02))
+  (wire (pts (xy 49.53 33.02) (xy 95.25 33.02))
+    (stroke (width 0) (type default))
+  )
+  (wire (pts (xy 200.66 151.13) (xy 53.34 151.13))
     (stroke (width 0) (type default))
   )
@@
     (stroke (width 0) (type default))
   )
-  (wire (pts (xy 53.34 52.07) (xy 73.66 52.07))
-    (stroke (width 0) (type default))
-  )
-  (wire (pts (xy 53.34 64.77) (xy 63.5 64.77))
+  (wire (pts (xy 49.53 52.07) (xy 73.66 52.07))
+    (stroke (width 0) (type default))
+  )
+  (wire (pts (xy 49.53 64.77) (xy 63.5 64.77))
     (stroke (width 0) (type default))
   )
@@
     (stroke (width 0) (type default))
   )
-  (wire (pts (xy 53.34 36.83) (xy 86.36 36.83))
+  (wire (pts (xy 49.53 36.83) (xy 86.36 36.83))
     (stroke (width 0) (type default))
   )
@@
     (stroke (width 0) (type default))
   )
+  (wire (pts (xy 203.2 106.68) (xy 200.66 106.68))
+    (stroke (width 0) (type default))
+  )
   (wire (pts (xy 121.92 30.48) (xy 203.2 30.48))
     (stroke (width 0) (type default))
@@
     (stroke (width 0) (type default))
   )
-  (wire (pts (xy 53.34 39.37) (xy 83.82 39.37))
+  (wire (pts (xy 49.53 39.37) (xy 83.82 39.37))
     (stroke (width 0) (type default))
   )
@@
     (stroke (width 0) (type default))
   )
-  (wire (pts (xy 53.34 49.53) (xy 76.2 49.53))
+  (wire (pts (xy 49.53 49.53) (xy 76.2 49.53))
     (stroke (width 0) (type default))
   )
@@
     (stroke (width 0) (type default))
   )
-  (wire (pts (xy 53.34 68.58) (xy 60.96 68.58))
+  (wire (pts (xy 49.53 68.58) (xy 60.96 68.58))
     (stroke (width 0) (type default))
   )
@@
     (stroke (width 0) (type default))
   )
-  (wire (pts (xy 53.34 62.23) (xy 66.04 62.23))
+  (wire (pts (xy 49.53 62.23) (xy 66.04 62.23))
+    (stroke (width 0) (type default))
+  )
+  (wire (pts (xy 200.66 106.68) (xy 200.66 151.13))
     (stroke (width 0) (type default))
   )
@@
     (stroke (width 0) (type default))
   )
-  (wire (pts (xy 53.34 43.18) (xy 81.28 43.18))
+  (wire (pts (xy 49.53 43.18) (xy 81.28 43.18))
     (stroke (width 0) (type default))
   )
@@
     (stroke (width 0) (type default))
   )
-  (wire (pts (xy 53.34 73.66) (xy 55.88 73.66))
+  (wire (pts (xy 49.53 73.66) (xy 55.88 73.66))
     (stroke (width 0) (type default))
   )
@@
     (stroke (width 0) (type default))
   )
+  (wire (pts (xy 53.34 151.13) (xy 53.34 76.2))
+    (stroke (width 0) (type default))
+  )
   (wire (pts (xy 92.71 92.71) (xy 92.71 111.76))
     (stroke (width 0) (type default))
   )
-  (wire (pts (xy 53.34 30.48) (xy 95.25 30.48))
+  (wire (pts (xy 49.53 30.48) (xy 95.25 30.48))
     (stroke (width 0) (type default))
   )
@@
     (stroke (width 0) (type default))
   )
-  (wire (pts (xy 58.42 71.12) (xy 53.34 71.12))
+  (wire (pts (xy 58.42 71.12) (xy 49.53 71.12))
     (stroke (width 0) (type default))
   )
@@
     (stroke (width 0) (type default))
   )
-  (wire (pts (xy 53.34 55.88) (xy 71.12 55.88))
+  (wire (pts (xy 49.53 55.88) (xy 71.12 55.88))
     (stroke (width 0) (type default))
   )
@@
     )
   )
-  (sheet (at 203.2 88.9) (size 38.1 17.78) (fields_autoplaced)
+  (sheet (at 203.2 88.9) (size 38.1 20.32) (fields_autoplaced)
     (stroke (width 0.1524) (type solid))
     (fill (color 0 0 0 0.0000))
@@
       (effects (font (size 1.27 1.27)) (justify left bottom))
     )
-    (property "Sheetfile" "sheets/filter-interface.kicad_sch" (at 203.2 107.2646 0)
+    (property "Sheetfile" "sheets/filter-interface.kicad_sch" (at 203.2 109.8046 0)
       (effects (font (size 1.27 1.27)) (justify left top) hide)
     )
@@
     )
     (pin "WAH_VELOCITY" output (at 203.2 104.14 180)
+      (effects (font (size 1.27 1.27)) (justify left))
+    )
+    (pin "FILTER_POSITION" output (at 203.2 106.68 180)
       (effects (font (size 1.27 1.27)) (justify left))
     )
@@
     )
   )
-  (sheet (at 26.67 27.94) (size 26.67 48.26) (fields_autoplaced)
+  (sheet (at 22.86 27.94) (size 26.67 50.8) (fields_autoplaced)
     (stroke (width 0.1524) (type solid))
     (fill (color 0 0 0 0.0000))
-    (property "Sheetname" "Digital" (at 26.67 27.2284 0)
+    (property "Sheetname" "Digital" (at 22.86 27.2284 0)
       (effects (font (size 1.27 1.27)) (justify left bottom))
     )
-    (property "Sheetfile" "sheets/digital.kicad_sch" (at 26.67 76.7846 0)
+    (property "Sheetfile" "sheets/digital.kicad_sch" (at 22.86 79.3246 0)
       (effects (font (size 1.27 1.27)) (justify left top) hide)
     )
-    (pin "RESET_4" output (at 53.34 49.53 0)
-      (effects (font (size 1.27 1.27)) (justify right))
-    )
-    (pin "AMP_4" output (at 53.34 52.07 0)
-      (effects (font (size 1.27 1.27)) (justify right))
-    )
-    (pin "RESET_5" output (at 53.34 55.88 0)
-      (effects (font (size 1.27 1.27)) (justify right))
-    )
-    (pin "AMP_5" output (at 53.34 58.42 0)
-      (effects (font (size 1.27 1.27)) (justify right))
-    )
-    (pin "RESET_6" output (at 53.34 62.23 0)
-      (effects (font (size 1.27 1.27)) (justify right))
-    )
-    (pin "AMP_6" output (at 53.34 64.77 0)
-      (effects (font (size 1.27 1.27)) (justify right))
-    )
-    (pin "RESET_2" output (at 53.34 36.83 0)
-      (effects (font (size 1.27 1.27)) (justify right))
-    )
-    (pin "AMP_2" output (at 53.34 39.37 0)
-      (effects (font (size 1.27 1.27)) (justify right))
-    )
-    (pin "RESET_3" output (at 53.34 43.18 0)
-      (effects (font (size 1.27 1.27)) (justify right))
-    )
-    (pin "AMP_3" output (at 53.34 45.72 0)
-      (effects (font (size 1.27 1.27)) (justify right))
-    )
-    (pin "RESET_1" output (at 53.34 30.48 0)
-      (effects (font (size 1.27 1.27)) (justify right))
-    )
-    (pin "AMP_1" output (at 53.34 33.02 0)
-      (effects (font (size 1.27 1.27)) (justify right))
-    )
-    (pin "ENVELOPE" output (at 53.34 68.58 0)
-      (effects (font (size 1.27 1.27)) (justify right))
-    )
-    (pin "FILTER_MOD" output (at 53.34 71.12 0)
-      (effects (font (size 1.27 1.27)) (justify right))
-    )
-    (pin "WAH_VELOCITY" input (at 53.34 73.66 0)
-      (effects (font (size 1.27 1.27)) (justify right))
-    )
+    (pin "RESET_4" output (at 49.53 49.53 0)
+      (effects (font (size 1.27 1.27)) (justify right))
+    )
+    (pin "AMP_4" output (at 49.53 52.07 0)
+      (effects (font (size 1.27 1.27)) (justify right))
+    )
+    (pin "RESET_5" output (at 49.53 55.88 0)
+      (effects (font (size 1.27 1.27)) (justify right))
+    )
+    (pin "AMP_5" output (at 49.53 58.42 0)
+      (effects (font (size 1.27 1.27)) (justify right))
+    )
+    (pin "RESET_6" output (at 49.53 62.23 0)
+      (effects (font (size 1.27 1.27)) (justify right))
+    )
+    (pin "AMP_6" output (at 49.53 64.77 0)
+      (effects (font (size 1.27 1.27)) (justify right))
+    )
+    (pin "RESET_2" output (at 49.53 36.83 0)
+      (effects (font (size 1.27 1.27)) (justify right))
+    )
+    (pin "AMP_2" output (at 49.53 39.37 0)
+      (effects (font (size 1.27 1.27)) (justify right))
+    )
+    (pin "RESET_3" output (at 49.53 43.18 0)
+      (effects (font (size 1.27 1.27)) (justify right))
+    )
+    (pin "AMP_3" output (at 49.53 45.72 0)
+      (effects (font (size 1.27 1.27)) (justify right))
+    )
+    (pin "RESET_1" output (at 49.53 30.48 0)
+      (effects (font (size 1.27 1.27)) (justify right))
+    )
+    (pin "AMP_1" output (at 49.53 33.02 0)
+      (effects (font (size 1.27 1.27)) (justify right))
+    )
+    (pin "ENVELOPE" output (at 49.53 68.58 0)
+      (effects (font (size 1.27 1.27)) (justify right))
+    )
+    (pin "FILTER_MOD" output (at 49.53 71.12 0)
+      (effects (font (size 1.27 1.27)) (justify right))
+    )
+    (pin "WAH_VELOCITY" input (at 49.53 73.66 0)
+      (effects (font (size 1.27 1.27)) (justify right))
+    )
+    (pin "EXTRA_ADC" input (at 49.53 76.2 0)
+      (effects (font (size 1.27 1.27)) (justify right))
+    )
