File: 1.1/schematics/control/sheets/mixer.kicad_sch (KiCad schematic)
At the start: 30 parts, among them U6 TL074

Commit message: Updated 1.1 mixer level
Parts:
- added C26, C27, C28: 470n (foil), Capacitor_THT:C_Rect_L7.0mm_W3.5mm_P5.00mm, symbol Device:C
- R20: value 100k -> 47k
- R21: value 100k -> 33k
Connections:
- net at R14.2, R15.2, R16.2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: now also C28.1; no longer C5.1, R21.1, U6.9 (-)
- net at R10.2, R11.2, R12.2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: now also C27.1; no longer C4.1, R20.1, U6.2 (-)
- new net: C28.2, C5.1, R21.1, U6.9 (-)
- new net: C27.2, C4.1, R20.1, U6.2 (-)
Other:
- moved on the sheet: R10, R11, R12, R13, R14, R15, R16, R17, R18, R19, R8, R9

Commit message: ✨ 1.1 Release
Hardware
- Fixes missing capacitor on the inputs of mixers. At f=0Hz the DCO's produce a DC output which shifts the center point of DCO's where f>0Hz. This happens on both the sawtooth and the squarewave output. A 470nF foil capacitor blocks all DC input on the input of the mixers.
- Decreases the aplification of mixers. The sum of 6 voices on both saw and square mixers are way too strong and hit the op-amp limits (+/-12V). The first stage of the mixers are reduced now to 1/3 on the squarewave and 1/2 on the sawtooth. Sounds much smoother!

Software
- Updates the MUX and the amp compensation output pin numbers according to the schematics.
Parts:
- removed C26: 470n (foil), Capacitor_THT:C_Rect_L7.0mm_W3.5mm_P5.00mm, symbol Device:C
Changed lines of the file:
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@@
-    )
-  )
-  (symbol (lib_id "Device:C") (at 107.95 80.01 90) (unit 1)
-    (in_bom yes) (on_board yes) (dnp no) (fields_autoplaced)
-    (property "Reference" "C26" (at 107.95 73.66 90)
-      (effects (font (size 1.27 1.27)))
-    )
-    (property "Value" "470n (foil)" (at 107.95 76.2 90)
-      (effects (font (size 1.27 1.27)))
-    )
-    (property "Footprint" "Capacitor_THT:C_Rect_L7.0mm_W3.5mm_P5.00mm" (at 111.76 79.0448 0)
-      (effects (font (size 1.27 1.27)) hide)
-    )
-    (property "Datasheet" "~" (at 107.95 80.01 0)
-      (effects (font (size 1.27 1.27)) hide)
-    )
-    (pin "1")
-    (pin "2")
-    (instances
-      (project "shmoergh-funk-live-control"
-        (path "/6d7b782d-8b2e-4b40-a99f-4bf41187d978/8c179049-6b29-46cf-9dc5-8ad32a25fc2f"
-          (reference "C26") (unit 1)
-        )
-      )
     )
   )
