File: 1.1/schematics/control/sheets/digital.kicad_sch (KiCad schematic)
At the start: 22 parts, among them U1 Pico, U3 TL072, U4 CD4051B, U5 MCP4822

Commit message: 1.1 changes
Connections:
- net Digital UI/EXTRA_GPIO1 renamed EXTRA_ADC
Changed lines of the file:
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@@
   (junction (at 35.56 74.93) (diameter 0) (color 0 0 0 0)
+  )
+  (junction (at 85.09 46.99) (diameter 0) (color 0 0 0 0)
   )
   (junction (at 57.15 177.8) (diameter 0) (color 0 0 0 0)
@@
     (stroke (width 0) (type default))
   )
+  (wire (pts (xy 85.09 46.99) (xy 92.71 46.99))
+    (stroke (width 0) (type default))
+  )
   (wire (pts (xy 83.82 29.21) (xy 83.82 41.91))
     (stroke (width 0) (type default))
@@
     (stroke (width 0) (type default))
   )
+  (wire (pts (xy 85.09 43.18) (xy 85.09 46.99))
+    (stroke (width 0) (type default))
+  )
   (wire (pts (xy 241.3 64.77) (xy 236.22 64.77))
     (stroke (width 0) (type default))
@@
     (stroke (width 0) (type default))
   )
+  (wire (pts (xy 88.9 43.18) (xy 85.09 43.18))
+    (stroke (width 0) (type default))
+  )
   (wire (pts (xy 254 48.26) (xy 260.35 48.26))
     (stroke (width 0) (type default))
@@
     (stroke (width 0) (type default))
   )
-  (wire (pts (xy 73.66 46.99) (xy 92.71 46.99))
+  (wire (pts (xy 73.66 46.99) (xy 85.09 46.99))
     (stroke (width 0) (type default))
   )
@@
     (effects (font (size 1.27 1.27)) (justify right))
   )
+  (hierarchical_label "EXTRA_ADC" (shape input) (at 88.9 43.18 0) (fields_autoplaced)
+    (effects (font (size 1.27 1.27)) (justify left))
+  )
   (hierarchical_label "AMP_3" (shape output) (at 80.01 69.85 0) (fields_autoplaced)
