File: 1.1/schematics/control/sheets/filter-interface.kicad_sch (KiCad schematic)
At the start: 10 parts

Commit message: 1.1 changes
Parts:
- added R62, R63, R64, R65: 100k, symbol Device:R
Connections:
- net +3.3V: now also #SW2.7, R62.1; no longer #SW2.10
- net GND: now also #SW2.11, R65.2; no longer #SW2.7, #SW2.8, #SW2.9
- net WAH_VELOCITY: no longer #SW2.14, J_FILTER_IO2.1 (Pin_1)
- new net: #SW2.8, R62.2, R63.1
- new net: #SW2.9, R63.2, R64.1
- new net: #SW2.10, R64.2, R65.1
- new net FILTER_POSITION: #SW2.14, J_FILTER_IO2.1 (Pin_1)
Other:
- note added: "FILTER_POSITION is connected to the (extra) ADC so that the MCU knows what the actual filter setting is."
- note removed: "WAH_VELOCITY is fed back to the MCU so that the amount of FILTER_DIGITAL_MOD can be calculated. 3.3V — Velocity ON 0 — Velocity OFF"
