File: 1.1/schematics/control/sheets/ui.kicad_sch (KiCad schematic)
At the start: 14 parts

Commit message: Added sound source UI
Parts:
- added SW1: SW_DPDT_x2, symbol Shmoergh_Custom_Components:SW_DPDT_x2
Changed lines of the file:
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@@
+    )
+  )
+  (symbol (lib_id "Shmoergh_Custom_Components:SW_DPDT_x2") (at 142.24 107.95 0) (unit 1)
+    (in_bom yes) (on_board yes) (dnp no) (fields_autoplaced)
+    (property "Reference" "SW1" (at 142.24 100.33 0)
+      (effects (font (size 1.27 1.27)))
+    )
+    (property "Value" "SW_DPDT_x2" (at 142.24 102.87 0)
+      (effects (font (size 1.27 1.27)))
+    )
+    (property "Footprint" "" (at 142.24 107.95 0)
+      (effects (font (size 1.27 1.27)) hide)
+    )
+    (property "Datasheet" "~" (at 142.24 107.95 0)
+      (effects (font (size 1.27 1.27)) hide)
+    )
+    (pin "1")
+    (pin "3")
+    (pin "5")
+    (pin "2")
+    (pin "4")
+    (pin "6")
+    (instances
+      (project "shmoergh-funk-live-control"
+        (path "/6d7b782d-8b2e-4b40-a99f-4bf41187d978/88d90181-522e-4756-bb1e-20cf1e1feb05/6fc25f0e-fad8-40a0-a83e-9226997ef918"
+          (reference "SW1") (unit 1)
+        )
+      )
     )
   )
@@
         )
       )
+    )
+  )
+  (symbol (lib_id "Shmoergh_Custom_Components:SW_DPDT_x2") (at 158.75 107.95 0) (unit 2)
+    (in_bom yes) (on_board yes) (dnp no) (fields_autoplaced)
+    (property "Reference" "SW1" (at 158.75 100.33 0)
+      (effects (font (size 1.27 1.27)))
+    )
+    (property "Value" "SW_DPDT_x2" (at 158.75 102.87 0)
+      (effects (font (size 1.27 1.27)))
+    )
+    (property "Footprint" "" (at 158.75 107.95 0)
+      (effects (font (size 1.27 1.27)) hide)
+    )
+    (property "Datasheet" "~" (at 158.75 107.95 0)
+      (effects (font (size 1.27 1.27)) hide)
+    )
+    (pin "1")
+    (pin "3")
+    (pin "5")
+    (pin "2")
+    (pin "4")
+    (pin "6")
+    (instances
+      (project "shmoergh-funk-live-control"
+        (path "/6d7b782d-8b2e-4b40-a99f-4bf41187d978/88d90181-522e-4756-bb1e-20cf1e1feb05/6fc25f0e-fad8-40a0-a83e-9226997ef918"
+          (reference "SW1") (unit 2)
+        )
+      )
