File: 1.0/schematics/control/sheets/filter-interface.kicad_sch (KiCad schematic)
At the start: 10 parts

Commit message: Updates to 1.0
Connections:
- net +3.3V: no longer #SW2.10
- net GND: now also #SW2.10; no longer #SW2.7, #SW2.8, #SW2.9
- no-connect marks 5 -> 8
Other:
- note added: "All this has to be wired on the panel."
- note added: "WAH_VELOCITY is fed back to the MCU so that the amount of FILTER_DIGITAL_MOD can be calculated. GND — Velocity ON NC — Velocity OFF"
- note removed: "All this has to be wired on the UI."
- note removed: "WAH_VELOCITY is fed back to the MCU so that the amount of FILTER_DIGITAL_MOD can be calculated. 3.3V — Velocity ON 0 — Velocity OFF"
Changed lines of the file:
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@@
   (junction (at 186.69 95.25) (diameter 0) (color 0 0 0 0)
   )
-  (junction (at 101.6 118.11) (diameter 0) (color 0 0 0 0)
-  )
   (junction (at 134.62 102.87) (diameter 0) (color 0 0 0 0)
   )
   (junction (at 175.26 95.25) (diameter 0) (color 0 0 0 0)
   )
-  (junction (at 101.6 115.57) (diameter 0) (color 0 0 0 0)
-  )
   (no_connect (at 107.95 125.73))
+  (no_connect (at 107.95 115.57))
+  (no_connect (at 107.95 113.03))
   (no_connect (at 107.95 123.19))
   (no_connect (at 223.52 113.03))
   (no_connect (at 107.95 107.95))
+  (no_connect (at 107.95 118.11))
   (no_connect (at 223.52 110.49))
   (wire (pts (xy 222.25 53.34) (xy 223.52 53.34))
@@
     (stroke (width 0) (type default))
   )
-  (wire (pts (xy 92.71 114.3) (xy 92.71 120.65))
-    (stroke (width 0) (type default))
-  )
   (wire (pts (xy 134.62 96.52) (xy 134.62 102.87))
     (stroke (width 0) (type default))
   )
-  (wire (pts (xy 101.6 118.11) (xy 101.6 115.57))
-    (stroke (width 0) (type default))
-  )
   (wire (pts (xy 149.86 68.58) (xy 186.69 68.58))
     (stroke (width 0) (type default))
@@
     (stroke (width 0) (type default))
   )
-  (wire (pts (xy 101.6 113.03) (xy 107.95 113.03))
-    (stroke (width 0) (type default))
-  )
   (wire (pts (xy 134.62 102.87) (xy 168.91 102.87))
     (stroke (width 0) (type default))
@@
     (stroke (width 0) (type default))
   )
-  (wire (pts (xy 107.95 118.11) (xy 101.6 118.11))
-    (stroke (width 0) (type default))
-  )
   (wire (pts (xy 184.15 107.95) (xy 186.69 107.95))
     (stroke (width 0) (type default))
@@
     (stroke (width 0) (type default))
   )
-  (wire (pts (xy 101.6 115.57) (xy 107.95 115.57))
-    (stroke (width 0) (type default))
-  )
   (wire (pts (xy 220.98 86.36) (xy 220.98 85.09))
     (stroke (width 0) (type default))
@@
     (stroke (width 0) (type default))
   )
-  (wire (pts (xy 101.6 115.57) (xy 101.6 113.03))
-    (stroke (width 0) (type default))
-  )
   (wire (pts (xy 222.25 49.53) (xy 222.25 53.34))
     (stroke (width 0) (type default))
@@
     (stroke (width 0) (type default))
   )
-  (wire (pts (xy 101.6 118.11) (xy 101.6 127))
-    (stroke (width 0) (type default))
-  )
   (wire (pts (xy 91.44 85.09) (xy 87.63 85.09))
     (stroke (width 0) (type default))
   )
-  (text "WAH_VELOCITY is fed back to the MCU\nso that the amount of FILTER_DIGITAL_MOD\ncan be calculated.\n3.3V — Velocity ON\n0 — Velocity OFF"
+  (text "WAH_VELOCITY is fed back to the MCU\nso that the amount of FILTER_DIGITAL_MOD\ncan be calculated.\nGND — Velocity ON\nNC — Velocity OFF"
     (at 132.08 135.89 0)
     (effects (font (size 1.27 1.27)) (justify left bottom))
@@
     (effects (font (size 1.27 1.27)) (justify left bottom))
   )
-  (text "All this has to be wired on the UI." (at 179.07 168.91 0)
+  (text "All this has to be wired on the panel." (at 179.07 168.91 0)
     (effects (font (size 1.27 1.27) (thickness 0.254) bold) (justify left bottom))
   )
@@
     )
   )
-  (symbol (lib_id "power:+3.3V") (at 92.71 114.3 0) (unit 1)
-    (in_bom yes) (on_board yes) (dnp no) (fields_autoplaced)
-    (property "Reference" "#PWR080" (at 92.71 118.11 0)
-      (effects (font (size 1.27 1.27)) hide)
-    )
-    (property "Value" "+3.3V" (at 92.71 110.49 0)
-      (effects (font (size 1.27 1.27)))
-    )
-    (property "Footprint" "" (at 92.71 114.3 0)
-      (effects (font (size 1.27 1.27)) hide)
-    )
-    (property "Datasheet" "" (at 92.71 114.3 0)
-      (effects (font (size 1.27 1.27)) hide)
-    )
-    (pin "1")
-    (instances
-      (project "shmoergh-funk-live-control"
-        (path "/6d7b782d-8b2e-4b40-a99f-4bf41187d978/5f1e1d4e-4c4f-4a8f-b34b-98240184a323"
-          (reference "#PWR080") (unit 1)
-        )
-      )
-    )
-  )
   (symbol (lib_id "power:+3.3V") (at 215.9 49.53 0) (unit 1)
     (in_bom yes) (on_board yes) (dnp no) (fields_autoplaced)
@@
     )
   )
-  (symbol (lib_id "power:GND") (at 101.6 127 0) (unit 1)
-    (in_bom yes) (on_board yes) (dnp no) (fields_autoplaced)
-    (property "Reference" "#PWR082" (at 101.6 133.35 0)
-      (effects (font (size 1.27 1.27)) hide)
-    )
-    (property "Value" "GND" (at 101.6 132.08 0)
-      (effects (font (size 1.27 1.27)))
-    )
-    (property "Footprint" "" (at 101.6 127 0)
-      (effects (font (size 1.27 1.27)) hide)
-    )
-    (property "Datasheet" "" (at 101.6 127 0)
-      (effects (font (size 1.27 1.27)) hide)
-    )
+  (symbol (lib_id "power:GND") (at 92.71 120.65 0) (unit 1)
+    (in_bom yes) (on_board yes) (dnp no) (fields_autoplaced)
+    (property "Reference" "#PWR082" (at 92.71 127 0)
+      (effects (font (size 1.27 1.27)) hide)
+    )
+    (property "Value" "GND" (at 92.71 125.73 0)
+      (effects (font (size 1.27 1.27)))
+    )
+    (property "Footprint" "" (at 92.71 120.65 0)
+      (effects (font (size 1.27 1.27)) hide)
+    )
+    (property "Datasheet" "" (at 92.71 120.65 0)
+      (effects (font (size 1.27 1.27)) hide)
+    )
