File: 1.0/schematics/control/sheets/lfo.kicad_sch (KiCad schematic)
At the start: 30 parts, among them Q1 BC548C, U10 TL072, U9 TL074

Commit message: Updates to 1.0
Parts:
- RV_LFO_SPEED1: value 100k -> A100k
Changed lines of the file:
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@@
   (symbol (lib_id "Device:R_Potentiometer") (at 52.07 54.61 0) (unit 1)
     (in_bom yes) (on_board yes) (dnp no) (fields_autoplaced)
-    (property "Reference" "RV_LFO_SPEED1" (at 49.53 53.975 0)
+    (property "Reference" "RV_LFO_SPEED1" (at 49.53 53.34 0)
       (effects (font (size 1.27 1.27)) (justify right))
     )
-    (property "Value" "100k" (at 49.53 56.515 0)
+    (property "Value" "A100k" (at 49.53 55.88 0)
       (effects (font (size 1.27 1.27)) (justify right))
     )
